File: pcb_files/ballanced_detector.sch (EAGLE design)
At the start: 70 parts, among them T1 TCM2-33X+, U1 HMC539ALP3EHCP_16_1_ADI-M, U2 ADA4961ACPZN-R7CP_24_7_ADI-M, U3 HMC539ALP3EHCP_16_1_ADI-M, U4 STM32L051K8T6LQFP32_7X7X1P4-M, U5 AS179-92LFSC70-6_SKY-M, U6 Value, U7 ADL8111ACCZNIC28_ADL8111ACCZN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, U8 TL7660CDGKTDGK8-M

Commit message: push before reboot
Connections:
- net ADC1: now also C11.1, R23.2, R24.1; no longer C10.1, R21.2, R22.1, R23.1
- net ADC2: now also C10.1, R21.2, R22.1, R23.1; no longer C11.1, R23.2, R24.1
Changed lines of the file:
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@@
 <part name="C2" library="adafruit" library_urn="urn:adsk.eagle:library:420" deviceset="C-US" device="C0402" package3d_urn="urn:adsk.eagle:package:6240340/1"/>
 <part name="C3" library="adafruit" library_urn="urn:adsk.eagle:library:420" deviceset="C-US" device="C0402" package3d_urn="urn:adsk.eagle:package:6240340/1" value="0.1uF"/>
-<part name="X1" library="adafruit" library_urn="urn:adsk.eagle:library:420" deviceset="SMACONNECTOR" device="_EDGE" package3d_urn="urn:adsk.eagle:package:6240945/1"/>
-<part name="X2" library="adafruit" library_urn="urn:adsk.eagle:library:420" deviceset="SMACONNECTOR" device="_EDGE" package3d_urn="urn:adsk.eagle:package:6240945/1"/>
+<part name="X1" library="adafruit" deviceset="SMACONNECTOR" device="_EDGE" package3d_urn="urn:adsk.eagle:package:6240945/1"/>
+<part name="X2" library="adafruit" deviceset="SMACONNECTOR" device="_EDGE" package3d_urn="urn:adsk.eagle:package:6240945/1"/>
 <part name="C4" library="adafruit" library_urn="urn:adsk.eagle:library:420" deviceset="C-US" device="C0402" package3d_urn="urn:adsk.eagle:package:6240340/1" value="0.1uF"/>
 <part name="T1" library="balun" deviceset="TCM2-33X+" device=""/>
-<part name="X3" library="adafruit" library_urn="urn:adsk.eagle:library:420" deviceset="SMACONNECTOR" device="_EDGE" package3d_urn="urn:adsk.eagle:package:6240945/1"/>
+<part name="X3" library="adafruit" deviceset="SMACONNECTOR" device="_EDGE" package3d_urn="urn:adsk.eagle:package:6240945/1"/>
 <part name="C5" library="adafruit" library_urn="urn:adsk.eagle:library:420" deviceset="C-US" device="C0402" package3d_urn="urn:adsk.eagle:package:6240340/1" value="330pF"/>
 <part name="C6" library="adafruit" library_urn="urn:adsk.eagle:library:420" deviceset="C-US" device="C0402" package3d_urn="urn:adsk.eagle:package:6240340/1" value="330pF"/>
@@
 <net name="ADC2" class="0">
 <segment>
-<pinref part="R23" gate="G$1" pin="2"/>
-<wire x1="-208.28" y1="-71.12" x2="-213.36" y2="-71.12" width="0.1524" layer="91"/>
-<pinref part="R24" gate="G$1" pin="1"/>
-<wire x1="-213.36" y1="-71.12" x2="-220.98" y2="-71.12" width="0.1524" layer="91"/>
-<wire x1="-220.98" y1="-71.12" x2="-220.98" y2="-73.66" width="0.1524" layer="91"/>
-<pinref part="C11" gate="G$1" pin="1"/>
-<wire x1="-213.36" y1="-73.66" x2="-213.36" y2="-71.12" width="0.1524" layer="91"/>
-<junction x="-213.36" y="-71.12"/>
-<label x="-220.98" y="-68.58" size="1.778" layer="95"/>
-</segment>
-<segment>
 <pinref part="U4" gate="A" pin="PA1"/>
 <wire x1="203.2" y1="-78.74" x2="190.5" y2="-78.74" width="0.1524" layer="91"/>
 <label x="185.42" y="-78.74" size="1.778" layer="95"/>
 </segment>
-</net>
-<net name="ADC1" class="0">
 <segment>
 <pinref part="R23" gate="G$1" pin="1"/>
@@
 <label x="-187.96" y="-68.58" size="1.778" layer="95"/>
 </segment>
+</net>
+<net name="ADC1" class="0">
 <segment>
 <pinref part="U4" gate="A" pin="PA0"/>
@@
 <label x="185.42" y="-76.2" size="1.778" layer="95"/>
 </segment>
-</net>
+<segment>
+<pinref part="R23" gate="G$1" pin="2"/>
+<wire x1="-208.28" y1="-71.12" x2="-213.36" y2="-71.12" width="0.1524" layer="91"/>
+<pinref part="R24" gate="G$1" pin="1"/>
+<wire x1="-213.36" y1="-71.12" x2="-220.98" y2="-71.12" width="0.1524" layer="91"/>
+<wire x1="-220.98" y1="-71.12" x2="-220.98" y2="-73.66" width="0.1524" layer="91"/>
+<pinref part="C11" gate="G$1" pin="1"/>
+<wire x1="-213.36" y1="-73.66" x2="-213.36" y2="-71.12" width="0.1524" layer="91"/>
+<junction x="-213.36" y="-71.12"/>
+<label x="-220.98" y="-68.58" size="1.778" layer="95"/>
+</segment>
+</net>
